File: kicad/logic-driver.kicad_sch (KiCad schematic)
At the start: 28 parts, among them J1 TIMEPULSE, J2 TIMEPULSE2, J3 LCD drive, J4 LCD bias, J5 LCD GND, J6 Photo GND, J7 Photo signal, Q1 HW5P-1, U1 4011, U2 4013, U3 4011, U4 TL074

Commit message: Adds rened kicad circuit and the kicad PCB design
Parts:
- removed C1: 1 uF, symbol Device:C
- removed J2: TIMEPULSE2, symbol Connector_Generic:Conn_01x01
- removed J4: LCD bias, symbol Connector_Generic:Conn_01x01
- removed J5: LCD GND, symbol Connector_Generic:Conn_01x01
- removed J6: Photo GND, symbol Connector_Generic:Conn_01x01
- removed R3: 47k, symbol Device:R_Trim
- removed R7: 1M, symbol Device:R
- removed unit 5 of U4
- added A1: Nucleo32-STM32G431, Module:Arduino_Nano, symbol MCU_Module:Arduino_Nano_Every
- added C1, C2: 2.2uF, Capacitor_THT:CP_Radial_D4.0mm_P1.50mm, symbol Device:C_Polarized_Small
- added C3: 100uF, Capacitor_THT:CP_Radial_D8.0mm_P2.50mm, symbol Device:C_Polarized
- added H1, H2, H3, H4: MountingHole, MountingHole:MountingHole_3.2mm_M3_ISO14580, symbol Mechanical:MountingHole
- added J10: LCD-B, Connector_PinSocket_2.54mm:PinSocket_1x02_P2.54mm_Vertical, symbol Connector_Generic:Conn_01x02
- added J2, J3: Power in, Connector_PinHeader_2.54mm:PinHeader_1x02_P2.54mm_Vertical, symbol Connector_Generic:Conn_01x02
- added J4: Onboard Neo_M8N, Neo-M8N_Module:Neo-M8N_1x05_P2.50mm_Horizontal, symbol Connector_Generic:Conn_01x05
- added J6: CN4, Connector_PinSocket_2.54mm:PinSocket_1x15_P2.54mm_Vertical, symbol Connector_Generic:Conn_01x15
- added J7: CN3, Connector_PinSocket_2.54mm:PinSocket_1x15_P2.54mm_Vertical, symbol Connector_Generic:Conn_01x15
- added J9: LCD-A, Connector_PinSocket_2.54mm:PinSocket_1x02_P2.54mm_Vertical, symbol Connector_Generic:Conn_01x02
- added JP1: +12V, Variants:TestPoint_Bridge_Pitch5.08mm_Drill0.7mm, symbol Jumper:Jumper_2_Open
- added JP2: +3V3, Variants:TestPoint_Bridge_Pitch5.08mm_Drill0.7mm, symbol Jumper:Jumper_2_Open
- added JP3: GND, Variants:TestPoint_Bridge_Pitch5.08mm_Drill0.7mm, symbol Jumper:Jumper_2_Open
- added JP4, JP6: Pos pulses, TestPoint:TestPoint_2Pads_Pitch2.54mm_Drill0.8mm, symbol Jumper:Jumper_2_Open
- added JP5, JP7: Neg pulses, TestPoint:TestPoint_2Pads_Pitch2.54mm_Drill0.8mm, symbol Jumper:Jumper_2_Open
- added RV1: 100k, Potentiometer_THT:Potentiometer_Vishay_T73XW_Horizontal, symbol Device:R_Potentiometer_Small
- added unit 2 of U2
- added unit 4 of U3
- added U4: LM7805_TO220, Package_TO_SOT_THT:TO-220-3_Vertical, symbol Regulator_Linear:LM7805_TO220
- added U6: ROB-14450, TB6612_Module_ROB-144450:TB6612_Module_ROB-14450, symbol TB6612_Motor_Driver_Module:ROB-14450
- D1: renamed from D2; footprint (none) -> LED_THT:LED_D5.0mm
- J1: value TIMEPULSE -> Neo-M8T; footprint (none) -> Connector_PinSocket_2.54mm:PinSocket_1x04_P2.54mm_Vertical; symbol Connector_Generic:Conn_01x01 -> Connector_Generic:Conn_01x04
- J5: renamed from J7; footprint (none) -> TestPoint:TestPoint_THTPad_D1.5mm_Drill0.7mm; symbol Connector_Generic:Conn_01x01 -> Connector_Generic:Conn_01x02
- J8: renamed from J3; value LCD drive -> LCD-opamp; footprint (none) -> Connector_PinSocket_2.54mm:PinSocket_1x02_P2.54mm_Vertical; symbol Connector_Generic:Conn_01x01 -> Connector_Generic:Conn_01x02
- R1: renamed from R8; footprint (none) -> Resistor_THT:R_Axial_DIN0207_L6.3mm_D2.5mm_P10.16mm_Horizontal
- R2: renamed from R9; footprint (none) -> Resistor_THT:R_Axial_DIN0207_L6.3mm_D2.5mm_P10.16mm_Horizontal
- R3: renamed from R1; footprint (none) -> Resistor_THT:R_Axial_DIN0207_L6.3mm_D2.5mm_P10.16mm_Horizontal
- R4: renamed from R2; value 82k -> 100k; footprint (none) -> Resistor_THT:R_Axial_DIN0207_L6.3mm_D2.5mm_P10.16mm_Horizontal
- R5: renamed from R4; footprint (none) -> Resistor_THT:R_Axial_DIN0207_L6.3mm_D2.5mm_P10.16mm_Horizontal
- R6: renamed from R5; footprint (none) -> Resistor_THT:R_Axial_DIN0207_L6.3mm_D2.5mm_P10.16mm_Horizontal
- R7: renamed from R6; footprint (none) -> Resistor_THT:R_Axial_DIN0207_L6.3mm_D2.5mm_P10.16mm_Horizontal
- TP1: renamed from TP2; footprint (none) -> TestPoint:TestPoint_THTPad_D1.5mm_Drill0.7mm
- TP2: renamed from TP1; footprint (none) -> TestPoint:TestPoint_THTPad_D1.5mm_Drill0.7mm
- TP3, TP4, TP5: footprint (none) -> TestPoint:TestPoint_THTPad_D1.5mm_Drill0.7mm
- U1, U2, U3: footprint (none) -> Package_DIP:CERDIP-14_W7.62mm_SideBrazed
- U5, U7: renamed from U4; value TL074 -> TL081; footprint (none) -> Package_DIP:CERDIP-8_W7.62mm_SideBrazed; symbol Amplifier_Operational:TL074 -> Amplifier_Operational:TL081
Connections:
- net +12V: now also A1.30 (VIN), J2.1 (Pin_1), J7.1 (Pin_1), JP1.1 (A), U6.1 (VM); no longer D1.2 (A)
- net +5V: now also D1.2 (A), C2.1, C3.1, U4.3 (VO)
- net GND: now also J5.2 (Pin_2), A1.29 (GND), A1.4 (GND), J2.2 (Pin_2), J4.4 (Pin_4), J6.4 (Pin_4), J7.2 (Pin_2), JP3.1 (A), U6.3 (GND), U6.8 (GND), U6.9 (GND); no longer U1.7 (VSS), U2.6 (S), U2.7 (VSS), U3.7 (VSS), U5.3 (+), U7.5 (+)
- net at TP2.1, U1.10, U3.1: now also U3.8; no longer U1.12
- net at U2.2 (~{Q}), U2.5 (D): now also U3.9; no longer U1.13
- net at R5.2, R6.2, R7.1: now also U7.2 (-); no longer U7.6 (-)
- net at R7.2, TP5.1: now also J8.1 (Pin_1), U7.6; no longer U7.7
- net at TP3.1, U3.4: now also JP4.1 (A); no longer R3.1
- net at Q1.2 (E), R2.1: now also J5.1 (Pin_1)
- net at U1.6, U2.3 (C): now also J1.3 (Pin_3)
- net at U5.1 (NULL): no longer R5.1
- net at R4.2: now also R5.1, U5.6
- new net: JP5.1 (A), TP4.1, U3.11
- new net: JP5.2 (B), R6.1
- new net: JP7.2 (B), U6.11 (BI2), U6.15 (AI2)
- new net: JP6.2 (B), U6.12 (BI1), U6.14 (AI1)
- new net: J9.1 (Pin_1), U6.4 (A01)
- new net: J9.2 (Pin_2), U6.5 (A02)
- new net: J10.2 (Pin_2), U6.6 (B02)
- new net: J10.1 (Pin_1), U6.7 (B01)
- new net: RV1.1, U7.1 (NULL)
- new net: RV1.3, U7.5 (NULL)
- new net: U3.10, U3.12, U3.13
- new net: JP4.2 (B), R3.1
- new net +L12V: C1.1, JP1.2 (B), U4.1 (VI), U5.7 (V+), U7.7 (V+)
- new net -L12V: J3.1 (Pin_1), RV1.2, U5.4 (V-), U7.4 (V-)
- new net AVDD: A1.18 (AREF), J7.13 (Pin_13)
- new net L3V3: J1.4 (Pin_4), JP2.2 (B)
- new net LGND: C1.2, C2.2, C3.2, J1.2 (Pin_2), J3.2 (Pin_2), J8.2 (Pin_2), JP3.2 (B), U1.7 (VSS), U2.6 (S), U2.7 (VSS), U3.7 (VSS), U4.2 (GND), U5.3 (+), U7.3 (+)
- new net MCU_3V3: A1.17 (3V3), J4.5 (Pin_5), J7.14 (Pin_14), JP2.1 (A)
- new net MCU_5V: A1.27 (+5V), J7.4 (Pin_4), U6.10 (PWMB), U6.13 (STBY), U6.16 (PWMA), U6.2 (VCC)
- new net NRSTA: A1.3 (~{RESET}), J6.3 (Pin_3)
- new net NRSTB: A1.28 (~{RESET}), J7.3 (Pin_3)
- new net PA0: A1.19 (A0), J7.12 (Pin_12)
- new net PA1: A1.20 (A1), J7.11 (Pin_11)
- new net PA10: A1.2 (RX1), J6.2 (Pin_2)
- new net PA11: A1.13 (D10), J4.3 (Pin_3), J6.13 (Pin_13)
- new net PA12: A1.5 (D2), J4.1 (Pin_1), J6.5 (Pin_5)
- new net PA15: A1.8 (D5), J6.8 (Pin_8)
- new net PA2: A1.26 (A7), J7.5 (Pin_5)
- new net PA3: A1.21 (A2), J7.10 (Pin_10)
- new net PA4: A1.22 (A3), J7.9 (Pin_9)
- new net PA5/PB7: A1.23 (SDA/A4), J7.8 (Pin_8)
- new net PA6/PA15: A1.24 (SCL/A5), J7.7 (Pin_7)
- new net PA7: A1.25 (A6), J7.6 (Pin_6)
- new net PA8: A1.12 (D9), J4.2 (Pin_2), J6.12 (Pin_12)
- new net PA9: A1.1 (TX1), J6.1 (Pin_1)
- new net PB0: A1.6 (D3), J6.6 (Pin_6), JP7.1 (A)
- new net PB3/PB8: A1.16 (SCK), J7.15 (Pin_15)
- new net PB4: A1.15 (MISO), J6.15 (Pin_15)
- new net PB5: A1.14 (MOSI), J6.14 (Pin_14)
- new net PB6: A1.9 (D6), J6.9 (Pin_9)
- new net PB7: A1.7 (D4), J6.7 (Pin_7), JP6.1 (A)
- new net PF0: A1.10 (D7), J6.10 (Pin_10)
- new net PF1: A1.11 (D8), J6.11 (Pin_11)
- now unconnected: U1.11
- no-connect marks 0 -> 11
Other:
- moved on the sheet: D1, Q1, R1, R2, R3, R4, R5, R6, R7, TP1, TP2, TP3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
